File: stabplate.sch (KiCad schematic (older format))
At the start: 7 parts, among them SW1 SW_Push, SW2 SW_Push, SW3 SW_Push, SW4 SW_Push, SW5 SW_Push, SW6 SW_Push, SW7 SW_Push

Commit message: changed to 2.75u, added copper planes
Parts:
- SW1, SW2, SW3, SW4: footprint MX_Only:MXOnly-2U-NoLED -> MX_Only:MXOnly-2.75U-NoLED
- SW5: footprint MX_Only:MXOnly-ISO-ROTATED-ReversedStabilizers-NoLED -> MX_Only:MXOnly-ISO
Changed lines of the file:
@@
 F 0 "SW2" H 2750 2685 50  0000 C CNN
 F 1 "SW_Push" H 2750 2594 50  0000 C CNN
-F 2 "MX_Only:MXOnly-2U-NoLED" H 2750 2600 50  0001 C CNN
+F 2 "MX_Only:MXOnly-2.75U-NoLED" H 2750 2600 50  0001 C CNN
 F 3 "~" H 2750 2600 50  0001 C CNN
 	1    2750 2400
@@
 F 0 "SW5" H 2750 3285 50  0000 C CNN
 F 1 "SW_Push" H 2750 3194 50  0000 C CNN
-F 2 "MX_Only:MXOnly-ISO-ROTATED-ReversedStabilizers-NoLED" H 2750 3200 50  0001 C CNN
+F 2 "MX_Only:MXOnly-ISO" H 2750 3200 50  0001 C CNN
 F 3 "~" H 2750 3200 50  0001 C CNN
 	1    2750 3000
@@
 F 0 "SW1" H 3825 2660 50  0000 C CNN
 F 1 "SW_Push" H 3825 2569 50  0000 C CNN
-F 2 "MX_Only:MXOnly-2U-NoLED" H 3825 2575 50  0001 C CNN
+F 2 "MX_Only:MXOnly-2.75U-NoLED" H 3825 2575 50  0001 C CNN
 F 3 "~" H 3825 2575 50  0001 C CNN
 	1    3825 2375
@@
 F 0 "SW4" H 3825 3260 50  0000 C CNN
 F 1 "SW_Push" H 3825 3169 50  0000 C CNN
-F 2 "MX_Only:MXOnly-2U-NoLED" H 3825 3175 50  0001 C CNN
+F 2 "MX_Only:MXOnly-2.75U-NoLED" H 3825 3175 50  0001 C CNN
 F 3 "~" H 3825 3175 50  0001 C CNN
 	1    3825 2975
@@
 F 0 "SW3" H 5400 2885 50  0000 C CNN
 F 1 "SW_Push" H 5400 2794 50  0000 C CNN
-F 2 "MX_Only:MXOnly-2U-NoLED" H 5400 2800 50  0001 C CNN
+F 2 "MX_Only:MXOnly-2.75U-NoLED" H 5400 2800 50  0001 C CNN
 F 3 "~" H 5400 2800 50  0001 C CNN
 	1    5400 2600
